File: sminchio.kicad_pcb (KiCad board)
At the start: 2 copper layers, 9 parts, among them J1 Screw_Terminal_01x06, Q1 SQ4435EY, Q2 SQ4435EY, U1 LTC4412xS6, U2 LTC4412xS6

Commit message: Almost complete version
Parts:
- added H1: MountingHole, Mounting_Holes:MountingHole_2.2mm_M2, F.Cu at (70.2, 62.9)
- added H2: MountingHole, Mounting_Holes:MountingHole_2.2mm_M2, F.Cu at (101.6, 62.9)
- added H3: MountingHole, Mounting_Holes:MountingHole_2.2mm_M2, F.Cu at (101.6, 94.6)
- added H4: MountingHole, Mounting_Holes:MountingHole_2.2mm_M2, F.Cu at (70.5, 94.6)
- added JP1: Jumper_2_Bridged, Pin_Headers:Pin_Header_Straight_1x02_Pitch2.54mm, F.Cu at (93.1, 78.6)
- moved R1 39.5 mm to (96.6, 83.8)
- moved D1 39.5 mm to (96.5, 85.7)
- moved R2 25.9 mm to (96.5, 74.3)
- moved D2 23.7 mm to (96.5, 72.4)
- moved U2 6.48 mm to (96.5, 68.6), turned to 270 degrees
- moved Q2 6.48 mm to (90.2, 68.6), turned to 0 degrees
- moved U1 2.84 mm to (96.5, 88.9)
- moved Q1 2.84 mm to (90.2, 88.9)
Connections:
- net Net-(J1-Pad6) renamed VIN_A
- J1 pad 1: GND -> VIN_B
- J1 pad 2: +12V -> GND
- J1 pad 4: Net-(J1-Pad4) -> +12V
- Q2 pad 5: Net-(J1-Pad4) -> VIN_B
- Q2 pad 6: Net-(J1-Pad4) -> VIN_B
- Q2 pad 7: Net-(J1-Pad4) -> VIN_B
- Q2 pad 8: Net-(J1-Pad4) -> VIN_B
- R1 pad 1: +12V -> Net-(D1-Pad1)
- R1 pad 2: Net-(D1-Pad2) -> Net-(JP1-Pad2)
- R2 pad 1: +12V -> Net-(JP1-Pad2)
- U1 pad 4: Net-(D1-Pad1) -> Net-(D1-Pad2)
- U2 pad 1: Net-(J1-Pad4) -> VIN_B
Routing:
- net Net-(JP1-Pad2): track 0.00 -> 13.7 mm
- net +12V: track 0.00 -> 11.7 mm
- net Net-(Q1-Pad4): track 0.00 -> 10.9 mm
- net Net-(Q2-Pad4): track 0.00 -> 6.81 mm
- net VIN_B: track 0.00 -> 6.44 mm
- net GND: track 0.00 -> 5.80 mm, vias 0 -> 2
- net Net-(D2-Pad1): track 0.00 -> 2.56 mm
- net Net-(D1-Pad1): track 0.00 -> 1.97 mm
- net Net-(D1-Pad2): track 0.00 -> 1.93 mm
- net Net-(D2-Pad2): track 0.00 -> 1.93 mm
- added copper zone on F.Cu, net +12V
- added copper zone on B.Cu, net GND
- added copper zone on F.Cu, net VIN_A
- added copper zone on F.Cu, net VIN_B
Other:
- board outline added: 36.6 x 37.1 mm
- board text added: "GND"
- board text added: "OUT"
- board text added: "Sminchio V1"
- board text added: "VA"
- board text added: "VB"
